File: 69.60784313725490196078431372549_Percent_keyboard.kicad_sch (KiCad schematic)
At the start: 5 parts, among them U1 ATMEGA32U4-AU

Commit message: reset push button, crystal
Parts:
- added C2, C3, C4: 0.1uF, symbol Device:C_Small
- added C5: 10uF, symbol Device:C_Small
- added C6, C7: 22pF, symbol Device:C_Small
- added R4: 10k, symbol Device:R_Small
- added SW1: SW_PUSH, symbol keyboard_parts:SW_PUSH
- added Y1: 16MHz, symbol Device:Crystal_GND24_Small
Connections:
- net +5V: now also U1.7 (VBUS), C2.1, C2.2, C3.1, C3.2, C4.1, C4.2, C5.1, C5.2, C6.2, C7.2, R4.1, SW1.1, Y1.2, Y1.4
- net D+: now reaches R2.2
- net D-: now reaches R3.2
- net at U1.13 (~{RESET}): now also R4.2, SW1.2
- net at U1.16 (XTAL2): now also C7.1, Y1.3
- net at U1.17 (XTAL1): now also C6.1, Y1.1

Commit message: Started switches, finished usb
Parts:
- added D0, D? (x13): D_Small, symbol Device:D_Small
- added F1: 500mA, symbol Device:Polyfuse_Small
- added SW0, SW? (x13): SW_DIP_x01, symbol Switch:SW_DIP_x01
- added USB1: Molex-0548190589, symbol random-keyboard-parts:Molex-0548190589
Connections:
- net +5V: now also F1.2
- net D+: now also USB1.3 (D+)
- net D-: now also USB1.4 (D-)
- new net: D?.2 (A), SW?.2 (x13)
- new net: D0.2 (A), SW0.2
- new net: D?.1 (K), D?.1 (K), D?.1 (K), D?.1 (K), D?.1 (K), D?.1 (K), D?.1 (K), D?.1 (K), D?.1 (K), D?.1 (K), D?.1 (K), D?.1 (K)
- new net GND: USB1.1 (GND)
- new net VCC: F1.1, USB1.5 (VBUS)

Commit message: Finished switches
Parts:
- added D10, D11, D13, D14, D15, D16, D17, D19, D2, D20, D21, D22, D24, D25, D26, D27, D28, D3, D30, D31, D32, D33, D34, D35, D36, D37, D39, D4, D40, D41, D42, D43, D45, D46, D47, D48, D49, D5, D51, D52, D53, D54, D55, D58, D59, D6, D60, D61, D62, D63, D64, D65, D66, D68, D69, D7, D70, D71, D72, D74, D75, D77, D78, D79, D8, D80, D81, D83, D84, D85, D86, D87, D9: D_Small, symbol Device:D_Small
- added SW10, SW11, SW13, SW14, SW15, SW16, SW17, SW19, SW2, SW20, SW21, SW22, SW25, SW26, SW27, SW28, SW29, SW3, SW31, SW32, SW33, SW34, SW35, SW36, SW37, SW38, SW4, SW40, SW41, SW42, SW43, SW44, SW46, SW47, SW48, SW49, SW5, SW50, SW52, SW53, SW54, SW55, SW56, SW59, SW6, SW60, SW61, SW62, SW63, SW64, SW65, SW66, SW67, SW69, SW7, SW70, SW71, SW72, SW73, SW75, SW76, SW78, SW79, SW8, SW80, SW81, SW82, SW84, SW85, SW86, SW87, SW88, SW9: SW_DIP_x01, symbol Switch:SW_DIP_x01
- gave numbers to parts that had none: 26
- renumbered C6 to C1, C7 to C2, C1 to C3, C2 to C4, C3 to C5, C4 to C6, C5 to C7, D0 to D56, R4 to R1, R1 to R2, R2 to R3, R3 to R4, SW1 to SW23, SW0 to SW57
Connections:
- net COL10: now reaches SW58.1
- net COL10: now also SW59.1, SW60.1, SW61.1, SW62.1
- net COL3: now reaches SW18.1
- net COL3: now also D15.1 (K), D21.1 (K), D26.1 (K), D32.1 (K), D36.1 (K), D4.1 (K), D41.1 (K), D47.1 (K), D53.1 (K), D60.1 (K), D64.1 (K), D70.1 (K), D79.1 (K), D85.1 (K), D9.1 (K), SW19.1, SW20.1, SW21.1, SW22.1
- net COL12: now reaches SW68.1
- net COL12: now also SW69.1, SW70.1, SW71.1, SW72.1, SW73.1
- net ROW0: now reaches D1.1 (K), D12.1 (K), D18.1 (K), D23.1 (K), D29.1 (K), D38.1 (K), D44.1 (K), D50.1 (K), D57.1 (K), D67.1 (K), D76.1 (K), D82.1 (K)
- net COL2: now reaches SW12.1
- net COL2: now also SW13.1, SW14.1, SW15.1, SW16.1, SW17.1
- net COL15: now reaches SW83.1
- net COL15: now also SW84.1, SW85.1, SW86.1, SW87.1, SW88.1
- net COL6: now reaches SW39.1
- net COL6: now also SW35.1, SW36.1, SW37.1, SW38.1, SW40.1, SW41.1, SW42.1, SW43.1, SW44.1
- net COL13: now reaches SW74.1
- net COL13: now also SW75.1, SW76.1
- net COL5: now reaches SW30.1
- net COL5: now also D11.1 (K), D28.1 (K), D43.1 (K), D55.1 (K), D6.1 (K), D66.1 (K), D72.1 (K), D81.1 (K), D87.1 (K), SW31.1, SW32.1, SW33.1, SW34.1
- net COL7: now reaches SW45.1
- net COL7: now also SW46.1, SW47.1, SW48.1, SW49.1, SW50.1
- net COL14: now reaches SW77.1
- net COL14: now also SW78.1, SW79.1, SW80.1, SW81.1, SW82.1
- net COL9: now reaches SW51.1
- net COL9: now also SW52.1, SW53.1, SW54.1, SW55.1, SW56.1
- net COL0: now reaches SW1.1
- net COL0: now also SW2.1, SW3.1, SW4.1, SW5.1, SW6.1
- net COL4: now reaches SW24.1
- net COL4: now also D10.1 (K), D16.1 (K), D22.1 (K), D27.1 (K), D37.1 (K), D42.1 (K), D48.1 (K), D5.1 (K), D54.1 (K), D61.1 (K), D65.1 (K), D71.1 (K), D80.1 (K), D86.1 (K), SW25.1, SW26.1, SW27.1, SW28.1, SW29.1
- new net: D32.2 (A), SW33.2
- new net: D27.2 (A), SW28.2
- new net: D48.2 (A), SW49.2
- new net: D15.2 (A), SW15.2
- new net: D35.2 (A), SW36.2
- new net: D59.2 (A), SW60.2
- new net: D54.2 (A), SW55.2
- new net: D51.2 (A), SW52.2
- new net: D79.2 (A), SW80.2
- new net: D43.2 (A), SW44.2
- new net: D11.2 (A), SW11.2
- new net: D86.2 (A), SW87.2
- new net: D47.2 (A), SW48.2
- new net: D20.2 (A), SW20.2
- new net: D46.2 (A), SW47.2
- new net: D72.2 (A), SW73.2
- new net: D30.2 (A), SW31.2
- new net: D26.2 (A), SW27.2
- new net: D63.2 (A), SW64.2
- new net: D78.2 (A), SW79.2
- new net: D62.2 (A), SW63.2
- new net: D10.2 (A), SW10.2
- new net: D2.2 (A), SW2.2
- new net: D4.2 (A), SW4.2
- new net: D52.2 (A), SW53.2
- new net: D84.2 (A), SW85.2
- new net: D87.2 (A), SW88.2
- new net: D80.2 (A), SW81.2
- new net: D68.2 (A), SW69.2
- new net: D7.2 (A), SW7.2
- new net: D55.2 (A), SW56.2
- new net: D42.2 (A), SW43.2
- new net: D58.2 (A), SW59.2
- new net: D37.2 (A), SW38.2
- new net: D34.2 (A), SW35.2
- new net: D49.2 (A), SW50.2
- new net: D39.2 (A), SW40.2
- new net: D14.2 (A), SW14.2
- new net: D81.2 (A), SW82.2
- new net: D3.2 (A), SW3.2
- new net: D77.2 (A), SW78.2
- new net: D5.2 (A), SW5.2
- new net: D19.2 (A), SW19.2
- new net: D13.2 (A), SW13.2
- new net: D31.2 (A), SW32.2
- new net: D40.2 (A), SW41.2
- new net: D45.2 (A), SW46.2
- new net: D17.2 (A), SW17.2
- new net: D74.2 (A), SW75.2
- new net: D60.2 (A), SW61.2
- new net: D61.2 (A), SW62.2
- new net: D85.2 (A), SW86.2
- new net: D9.2 (A), SW9.2
- new net: D36.2 (A), SW37.2
- new net: D53.2 (A), SW54.2
- new net: D71.2 (A), SW72.2
- new net: D83.2 (A), SW84.2
- new net: D28.2 (A), SW29.2
- new net: D69.2 (A), SW70.2
- new net: D64.2 (A), SW65.2
- new net: D21.2 (A), SW21.2
- new net: D25.2 (A), SW26.2
- new net: D22.2 (A), SW22.2
- new net: D66.2 (A), SW67.2
- new net: D8.2 (A), SW8.2
- new net: D6.2 (A), SW6.2
- new net: D41.2 (A), SW42.2
- new net: D75.2 (A), SW76.2
- new net: D16.2 (A), SW16.2
- new net: D65.2 (A), SW66.2
- new net: D24.2 (A), SW25.2
- new net: D70.2 (A), SW71.2
- new net: D33.2 (A), SW34.2
- new net COL1: SW10.1, SW11.1, SW7.1, SW8.1, SW9.1
- new net COL11: SW63.1, SW64.1, SW65.1, SW66.1, SW67.1
- new net ROW1: D13.1 (K), D19.1 (K), D2.1 (K), D24.1 (K), D30.1 (K), D34.1 (K), D39.1 (K), D45.1 (K), D51.1 (K), D62.1 (K), D68.1 (K), D7.1 (K), D74.1 (K), D77.1 (K), D83.1 (K)
- new net ROW2: D14.1 (K), D20.1 (K), D25.1 (K), D3.1 (K), D31.1 (K), D35.1 (K), D40.1 (K), D46.1 (K), D52.1 (K), D59.1 (K), D63.1 (K), D69.1 (K), D75.1 (K), D78.1 (K), D8.1 (K), D84.1 (K)

Commit message: started adding footprints
Parts:
- C1, C2, C3, C4, C5, C6, C7: footprint (none) -> Capacitor_SMD:C_0805_2012Metric
- D1, D10, D11, D12, D13, D14, D15, D16, D17, D18, D19, D2, D20, D21, D22, D23, D24, D25, D26, D27, D28, D29, D3, D30, D31, D32, D33, D34, D35, D36, D37, D38, D39, D4, D40, D41, D42, D43, D44, D45, D46, D47, D48, D49, D5, D50, D51, D52, D53, D54, D55, D56, D57, D58, D59, D6, D60, D61, D62, D63, D64, D65, D66, D67, D68, D69, D7, D70, D71, D72, D73, D74, D75, D76, D77, D78, D79, D8, D80, D81, D82, D83, D84, D85, D86, D87, D9: footprint (none) -> Diode_SMD:D_SOD-123
- Y1: footprint (none) -> Fuse:Fuse_1206_3216Metric

Commit message: add kicad libraries finished footprints started PCB
Parts:
- removed D56, D62, D63, D64, D65, D66: D_Small, Diode_SMD:D_SOD-123, symbol Device:D_Small
- removed SW57, SW63, SW64, SW65, SW66, SW67: SW_DIP_x01, symbol Switch:SW_DIP_x01
- F1: footprint (none) -> Fuse:Fuse_1206_3216Metric
- R1, R2, R3, R4: footprint (none) -> Resistor_SMD:R_0805_2012Metric
- SW1, SW10, SW12, SW13, SW14, SW15, SW16, SW18, SW19, SW2, SW20, SW21, SW22, SW24, SW25, SW26, SW27, SW28, SW30, SW31, SW32, SW33, SW34, SW35, SW36, SW37, SW38, SW39, SW40, SW41, SW42, SW43, SW45, SW46, SW47, SW48, SW49, SW51, SW52, SW53, SW54, SW55, SW58, SW59, SW60, SW61, SW62, SW68, SW69, SW7, SW70, SW71, SW74, SW75, SW76, SW77, SW8, SW81, SW83, SW84, SW85, SW86, SW87, SW88, SW9: footprint (none) -> CherryMX_KailhSocket_LED:CherryMX_1.00u_KailhSocket_LED
- SW11, SW17, SW44, SW50, SW56, SW6, SW82: footprint (none) -> CherryMX_KailhSocket_LED:CherryMX_1.25u_KailhSocket_LED
- SW29: footprint (none) -> CherryMX_KailhSocket_LED:CherryMX_6.00u_KailhSocket_LED
- SW3, SW79: footprint (none) -> CherryMX_KailhSocket_LED:CherryMX_1.50u_KailhSocket_LED
- SW4, SW73: footprint (none) -> CherryMX_KailhSocket_LED:CherryMX_1.75u_KailhSocket_LED
- SW5, SW72, SW78: footprint (none) -> CherryMX_KailhSocket_LED:CherryMX_2.00u_KailhSocket_LED
- SW80: footprint (none) -> CherryMX_KailhSocket_LED:CherryMX_2.25u_KailhSocket_LED
- USB1: footprint (none) -> random-keyboard-parts:Molex-0548190589

Commit message: Recommit 12-03-2022
Connections:
- net COL0: now also U1.30 (PB6)
- net COL1: now also U1.12 (PB7)
- net COL10: now also U1.32 (PC7)
- net COL12: now also U1.36 (PF7)
- net COL13: now also U1.37 (PF6)
- net COL14: now also U1.38 (PF5)
- net COL15: now also U1.39 (PF4)
- net COL2: now also U1.18 (PD0)
- net COL3: now also U1.19 (PD1)
- net COL4: now also U1.20 (PD2)
- net COL5: now also U1.21 (PD3)
- net COL6: now also U1.25 (PD4)
- net COL7: now also U1.22 (PD5)
- net COL9: now also U1.27 (PD7)
- net ROW0: now also U1.8 (PB0)
- net ROW1: now also U1.9 (PB1)
- net ROW2: now also U1.10 (PB2)
- net COL11: now reaches U1.1 (PE6)
- net ROW3: now reaches U1.11 (PB3)
- net COL8: now reaches U1.26 (PD6)
- net ROW4: now reaches U1.28 (PB4)
- net ROW5: now reaches U1.29 (PB5)
Other:
- moved on the sheet: C1, C2, C3, C4, C5, C6, C7, D1, D10, D11, D12, D13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
